File: opamps.sch (KiCad schematic (older format))
At the start: 41 parts

Commit message: passed schematic review
Parts:
- L? (x3): value TM_L -> 10uH
Changed lines of the file:
@@
 P 7500 1800
 F 0 "L?" V 7400 1800 50  0000 C CNN
-F 1 "TM_L" V 7550 1805 50  0000 C CNN
+F 1 "10uH" V 7550 1805 50  0000 C CNN
 F 2 "" H 7500 1805 60  0000 C CNN
 F 3 "" H 7500 1805 60  0000 C CNN
@@
 P 2400 1800
 F 0 "L?" V 2300 1800 50  0000 C CNN
-F 1 "TM_L" V 2450 1805 50  0000 C CNN
+F 1 "10uH" V 2450 1805 50  0000 C CNN
 F 2 "" H 2400 1805 60  0000 C CNN
 F 3 "" H 2400 1805 60  0000 C CNN
@@
 P 12700 1800
 F 0 "L?" V 12600 1800 50  0000 C CNN
-F 1 "TM_L" V 12750 1805 50  0000 C CNN
+F 1 "10uH" V 12750 1805 50  0000 C CNN
 F 2 "" H 12700 1805 60  0000 C CNN
 F 3 "" H 12700 1805 60  0000 C CNN
