File: opamps.sch (KiCad schematic (older format))
At the start: 41 parts

Commit message: added testpoint part number, small net naming changes
Parts:
- TP? (x9): value TP -> 0914-0-15-20-77-14-11-0
Changed lines of the file:
@@
 P 7300 3400
 F 0 "TP?" H 7300 3450 60  0000 C CNN
-F 1 "TP" H 7300 3350 60  0001 C CNN
+F 1 "0914-0-15-20-77-14-11-0" H 7300 3350 60  0001 C CNN
 F 2 "" H 7300 3400 60  0000 C CNN
 F 3 "" H 7300 3400 60  0000 C CNN
@@
 P 7100 3400
 F 0 "TP?" H 7100 3450 60  0000 C CNN
-F 1 "TP" H 7100 3350 60  0001 C CNN
+F 1 "0914-0-15-20-77-14-11-0" H 7100 3350 60  0001 C CNN
 F 2 "" H 7100 3400 60  0000 C CNN
 F 3 "" H 7100 3400 60  0000 C CNN
@@
 P 7300 6500
 F 0 "TP?" H 7300 6550 60  0000 C CNN
-F 1 "TP" H 7300 6450 60  0001 C CNN
+F 1 "0914-0-15-20-77-14-11-0" H 7300 6450 60  0001 C CNN
 F 2 "" H 7300 6500 60  0000 C CNN
 F 3 "" H 7300 6500 60  0000 C CNN
@@
 P 7100 6500
 F 0 "TP?" H 7100 6550 60  0000 C CNN
-F 1 "TP" H 7100 6450 60  0001 C CNN
+F 1 "0914-0-15-20-77-14-11-0" H 7100 6450 60  0001 C CNN
 F 2 "" H 7100 6500 60  0000 C CNN
 F 3 "" H 7100 6500 60  0000 C CNN
@@
 P 3000 6800
 F 0 "TP?" H 3000 6850 60  0000 C CNN
-F 1 "TP" H 3000 6750 60  0001 C CNN
+F 1 "0914-0-15-20-77-14-11-0" H 3000 6750 60  0001 C CNN
 F 2 "" H 3000 6800 60  0000 C CNN
 F 3 "" H 3000 6800 60  0000 C CNN
@@
 P 3000 8000
 F 0 "TP?" H 3000 8050 60  0000 C CNN
-F 1 "TP" H 3000 7950 60  0001 C CNN
+F 1 "0914-0-15-20-77-14-11-0" H 3000 7950 60  0001 C CNN
 F 2 "" H 3000 8000 60  0000 C CNN
 F 3 "" H 3000 8000 60  0000 C CNN
@@
 P 2200 3400
 F 0 "TP?" H 2200 3450 60  0000 C CNN
-F 1 "TP" H 2200 3350 60  0001 C CNN
+F 1 "0914-0-15-20-77-14-11-0" H 2200 3350 60  0001 C CNN
 F 2 "" H 2200 3400 60  0000 C CNN
 F 3 "" H 2200 3400 60  0000 C CNN
@@
 P 2000 3400
 F 0 "TP?" H 2000 3450 60  0000 C CNN
-F 1 "TP" H 2000 3350 60  0001 C CNN
+F 1 "0914-0-15-20-77-14-11-0" H 2000 3350 60  0001 C CNN
 F 2 "" H 2000 3400 60  0000 C CNN
 F 3 "" H 2000 3400 60  0000 C CNN
@@
 P 12500 3400
 F 0 "TP?" H 12500 3450 60  0000 C CNN
-F 1 "TP" H 12500 3350 60  0001 C CNN
+F 1 "0914-0-15-20-77-14-11-0" H 12500 3350 60  0001 C CNN
 F 2 "" H 12500 3400 60  0000 C CNN
 F 3 "" H 12500 3400 60  0000 C CNN

Commit message: annotated
Parts:
- gave numbers to parts that had none: 29

Commit message: annotated, netlist
Connections:
- wire segments 218 -> 167

Commit message: components and footprints
Parts:
- C501, C502, C503, C504, C505, C506, C507, C508, C509: footprint (none) -> tm-kicad-lib:SMD-0402-C
- L501, L502, L503: footprint (none) -> tm-kicad-lib:SMD-0603-R
- RN501, RN502, RN503, RN504: footprint (none) -> tm-kicad-lib:ACAS0612
- TP501, TP502, TP503, TP504, TP505, TP506, TP507, TP508, TP509: value 0914-0-15-20-77-14-11-0 -> 0932-0-15-20-77-14-11-0
- TP510: footprint (none) -> tm-kicad-lib:Testpoint
- U501, U502, U503: footprint (none) -> SMD_Packages:SOIC-14_N

Commit message: swapped testpoints
Parts:
- TP501, TP502, TP503, TP504, TP505, TP506, TP507, TP508, TP509: footprint (none) -> tm-kicad-lib:0932-0-15-20-77-14-11-0
Changed lines of the file:
@@
 F 0 "TP507" H 7300 3450 60  0000 C CNN
 F 1 "0932-0-15-20-77-14-11-0" H 7300 3350 60  0001 C CNN
-F 2 "" H 7300 3400 60  0001 C CNN
+F 2 "tm-kicad-lib:0932-0-15-20-77-14-11-0" H 7300 3400 60  0001 C CNN
 F 3 "" H 7300 3400 60  0000 C CNN
 	1    7300 3400
@@
 F 0 "TP505" H 7100 3450 60  0000 C CNN
 F 1 "0932-0-15-20-77-14-11-0" H 7100 3350 60  0001 C CNN
-F 2 "" H 7100 3400 60  0001 C CNN
+F 2 "tm-kicad-lib:0932-0-15-20-77-14-11-0" H 7100 3400 60  0001 C CNN
 F 3 "" H 7100 3400 60  0000 C CNN
 	1    7100 3400
@@
 F 0 "TP508" H 7300 6550 60  0000 C CNN
 F 1 "0932-0-15-20-77-14-11-0" H 7300 6450 60  0001 C CNN
-F 2 "" H 7300 6500 60  0001 C CNN
+F 2 "tm-kicad-lib:0932-0-15-20-77-14-11-0" H 7300 6500 60  0001 C CNN
 F 3 "" H 7300 6500 60  0000 C CNN
 	1    7300 6500
@@
 F 0 "TP506" H 7100 6550 60  0000 C CNN
 F 1 "0932-0-15-20-77-14-11-0" H 7100 6450 60  0001 C CNN
-F 2 "" H 7100 6500 60  0001 C CNN
+F 2 "tm-kicad-lib:0932-0-15-20-77-14-11-0" H 7100 6500 60  0001 C CNN
 F 3 "" H 7100 6500 60  0000 C CNN
 	1    7100 6500
@@
 F 0 "TP503" H 3000 6850 60  0000 C CNN
 F 1 "0932-0-15-20-77-14-11-0" H 3000 6750 60  0001 C CNN
-F 2 "" H 3000 6800 60  0001 C CNN
+F 2 "tm-kicad-lib:0932-0-15-20-77-14-11-0" H 3000 6800 60  0001 C CNN
 F 3 "" H 3000 6800 60  0000 C CNN
 	1    3000 6800
@@
 F 0 "TP504" H 3000 8050 60  0000 C CNN
 F 1 "0932-0-15-20-77-14-11-0" H 3000 7950 60  0001 C CNN
-F 2 "" H 3000 8000 60  0001 C CNN
+F 2 "tm-kicad-lib:0932-0-15-20-77-14-11-0" H 3000 8000 60  0001 C CNN
 F 3 "" H 3000 8000 60  0000 C CNN
 	1    3000 8000
@@
 F 0 "TP502" H 2200 3450 60  0000 C CNN
 F 1 "0932-0-15-20-77-14-11-0" H 2200 3350 60  0001 C CNN
-F 2 "" H 2200 3400 60  0001 C CNN
+F 2 "tm-kicad-lib:0932-0-15-20-77-14-11-0" H 2200 3400 60  0001 C CNN
 F 3 "" H 2200 3400 60  0000 C CNN
 	1    2200 3400
@@
 F 0 "TP501" H 2000 3450 60  0000 C CNN
 F 1 "0932-0-15-20-77-14-11-0" H 2000 3350 60  0001 C CNN
-F 2 "" H 2000 3400 60  0001 C CNN
+F 2 "tm-kicad-lib:0932-0-15-20-77-14-11-0" H 2000 3400 60  0001 C CNN
 F 3 "" H 2000 3400 60  0000 C CNN
 	1    2000 3400
@@
 F 0 "TP509" H 12500 3450 60  0000 C CNN
 F 1 "0932-0-15-20-77-14-11-0" H 12500 3350 60  0001 C CNN
-F 2 "" H 12500 3400 60  0001 C CNN
+F 2 "tm-kicad-lib:0932-0-15-20-77-14-11-0" H 12500 3400 60  0001 C CNN
 F 3 "" H 12500 3400 60  0000 C CNN
 	1    12500 3400

Commit message: on to layout! and what an adventure it will be...
Parts:
- removed TP501, TP502, TP506, TP508: 0932-0-15-20-77-14-11-0, tm-kicad-lib:0932-0-15-20-77-14-11-0, symbol TP
Connections:
- wire segments 167 -> 163
Other:
- moved on the sheet: U501A, U501B, U501C, U501D, U501E, U502A, U502B, U502C, U502D, U502E, U503A, U503B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
